File: HotplateController/HotplateController.kicad_sch (KiCad schematic)
At the start: 22 parts

Commit message: Added fab outputs, prep for pcbway contest
Parts:
- removed C?: 0.1u, Capacitor_SMD:C_0603_1608Metric_Pad1.08x0.95mm_HandSolder, symbol Device:C
- removed R? (x5): 10k, Resistor_SMD:R_0603_1608Metric_Pad0.98x0.95mm_HandSolder, symbol Device:R_US
- removed SW?: RotaryEncoder_Switch, Rotary_Encoder:RotaryEncoder_Alps_EC11E-Switch_Vertical_H20mm, symbol Device:RotaryEncoder_Switch
- added C1: 0.01u, Capacitor_SMD:C_0603_1608Metric, symbol Device:C
- added C10, C2, C7, C8, C9: 0.1u, Capacitor_SMD:C_0603_1608Metric, symbol Device:C
- added C3: 10u, Capacitor_SMD:C_0805_2012Metric_Pad1.18x1.45mm_HandSolder, symbol Device:C
- added H1, H2, H3, H4: MountingHole_Pad, MountingHole:MountingHole_3.2mm_M3_ISO7380_Pad, symbol Mechanical:MountingHole_Pad
- added J1, J5: Conn_01x02, TerminalBlock_MetzConnect:TerminalBlock_MetzConnect_Type086_RT03402HBLC_1x02_P3.81mm_Horizontal, symbol Connector_Generic:Conn_01x02
- added R1, R2, R6, R7, R8: 0, Resistor_SMD:R_0603_1608Metric_Pad0.98x0.95mm_HandSolder, symbol Device:R_US
- added R3, R4: 10k, Resistor_SMD:R_0603_1608Metric_Pad0.98x0.95mm_HandSolder, symbol Device:R_US
- added SW1, SW2, SW3, SW4: SW_Push, Button_Switch_THT:SW_PUSH_6mm, symbol Switch:SW_Push
- added U1: MAX31855KASA, Package_SO:SOIC-8_3.9x4.9mm_P1.27mm, symbol Sensor_Temperature:MAX31855KASA
- J2: renamed from J?; footprint (none) -> Connector_PinHeader_2.54mm:PinHeader_1x04_P2.54mm_Vertical
- J3, J4: renamed from J?; footprint (none) -> Connector_PinHeader_2.54mm:PinHeader_1x02_P2.54mm_Vertical
- gave numbers to parts that had none: 12
Connections:
- net +3V3: now also C2.1, C3.2, R3.1, R4.1, U1.4 (VCC)
- net +5V: now also J5.1 (Pin_1)
- net GND: now also C10.2, C2.2, C3.1, C7.2, C8.2, C9.2, H1.1, H2.1, H3.1, H4.1, J5.2 (Pin_2), SW1.1, SW2.1, SW3.1, SW4.1, U1.1 (GND)
- net SSR_OUT: now also U2.21 (GPIO16); no longer U2.26 (GPIO20)
- net TEMP_IN: now also U2.34 (GPIO28_ADC2); no longer U2.31 (GPIO26_ADC0)
- net SPI_SCLK: now reaches U2.14 (GPIO10)
- net SPI_SCLK: now also R6.1
- net SPI_DATA: now reaches U2.16 (GPIO12)
- net SPI_DATA: now also R7.1
- net SPI_CSN: now reaches U2.17 (GPIO13)
- net SPI_CSN: now also R8.1
- net SW_DWN: now reaches U2.20 (GPIO15)
- net SW_DWN: now also C9.1, SW3.2
- net SW_RUN: now reaches U2.30 (RUN)
- net SW_RUN: now also C10.1, SW4.2
- net ENC_A renamed SW_UP
- net SW_UP: now also C7.1, SW1.2
- net ENC_B renamed SW_SEL
- net SW_SEL: now also C8.1, SW2.2
- net ENC_SW: no longer names the net of U2.10 (GPIO7)
- new net KTTC_N: C1.2, R2.2, U1.2 (T-)
- new net KTTC_N_R: J1.2 (Pin_2), R2.1
- new net KTTC_P: C1.1, R1.2, U1.3 (T+)
- new net KTTC_P_R: J1.1 (Pin_1), R1.1
- new net SPI_CSN_R: R4.2, R8.2, U1.6 (~{CS})
- new net SPI_DATA_R: R7.2, U1.7 (SO)
- new net SPI_SCLK_R: R3.2, R6.2, U1.5 (SCK)
- no-connect marks 0 -> 17
Other:
- note added: "5V IN FROM AC-5V CONVERTER 3V3 SUPPLY FOR BOARD FROM PICO"
- note added: "CHECK THAT PINOUT OF DISPLAY IS CONSISTENT WITH LISTED HERE PULL-UPS MAY BE OPTIONAL"
- note added: "OPTIONAL THERMOCOUPLE INPUT AND THERMOCOUPLE AMP"
- company: (none) -> HAPPY LITTLE PCBS
- title: (none) -> HOTPLATE CONTROLLER
- moved on the sheet: C4, C5, C6, D1, J2, J3, J4, R10, R11, R12, R13, R14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
